File: mfk5.kicad_pcb (KiCad board)
At the start: 2 copper layers, 84.5 x 57.2 mm, 18 parts, among them SW1 RST, SW2 COL1_ROW1, SW3 COL2_ROW1, SW4 COL1_ROW2, SW5 COL2_ROW2, SW6 COL1_ROW3, U1 Pro Micro

Commit message: Update mfk5 layout.
Other:
- board text added: "mfk5 rev. 2 @niw"
- board text removed: "mfk5 rev. 1 @niw"
Changed lines of the file:
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@@
     (fp_rect (start -7 -7) (end 7 7)
       (stroke (width 0.05) (type solid)) (fill none) (layer "Dwgs.User"))
-    (fp_line (start -15.5 7.2) (end -15.5 -9.2)
-      (stroke (width 0.15) (type default)) (layer "Edge.Cuts"))
-    (fp_line (start -15.2 -9.5) (end -8.8 -9.5)
-      (stroke (width 0.15) (type default)) (layer "Edge.Cuts"))
-    (fp_line (start -8.8 7.5) (end -15.2 7.5)
-      (stroke (width 0.15) (type default)) (layer "Edge.Cuts"))
-    (fp_line (start -8.5 -9.2) (end -8.5 7.2)
-      (stroke (width 0.15) (type default)) (layer "Edge.Cuts"))
-    (fp_line (start 8.5 7.2) (end 8.5 -9.2)
-      (stroke (width 0.15) (type default)) (layer "Edge.Cuts"))
-    (fp_line (start 8.8 -9.5) (end 15.2 -9.5)
-      (stroke (width 0.15) (type default)) (layer "Edge.Cuts"))
-    (fp_line (start 15.2 7.5) (end 8.8 7.5)
-      (stroke (width 0.15) (type default)) (layer "Edge.Cuts"))
-    (fp_line (start 15.5 -9.2) (end 15.5 7.2)
-      (stroke (width 0.15) (type default)) (layer "Edge.Cuts"))
-    (fp_arc (start -15.5 -9.2) (mid -15.412132 -9.412132) (end -15.2 -9.5)
-      (stroke (width 0.15) (type default)) (layer "Edge.Cuts"))
-    (fp_arc (start -15.2 7.5) (mid -15.412132 7.412132) (end -15.5 7.2)
-      (stroke (width 0.15) (type default)) (layer "Edge.Cuts"))
-    (fp_arc (start -8.8 -9.5) (mid -8.587868 -9.412132) (end -8.5 -9.2)
-      (stroke (width 0.15) (type default)) (layer "Edge.Cuts"))
-    (fp_arc (start -8.5 7.2) (mid -8.587868 7.412132) (end -8.8 7.5)
-      (stroke (width 0.15) (type default)) (layer "Edge.Cuts"))
-    (fp_arc (start 8.5 -9.2) (mid 8.587868 -9.412132) (end 8.8 -9.5)
-      (stroke (width 0.15) (type default)) (layer "Edge.Cuts"))
-    (fp_arc (start 8.8 7.5) (mid 8.587868 7.412132) (end 8.5 7.2)
-      (stroke (width 0.15) (type default)) (layer "Edge.Cuts"))
-    (fp_arc (start 15.2 -9.5) (mid 15.412132 -9.412132) (end 15.5 -9.2)
-      (stroke (width 0.15) (type default)) (layer "Edge.Cuts"))
-    (fp_arc (start 15.5 7.2) (mid 15.412132 7.412132) (end 15.2 7.5)
+    (fp_line (start -15.5 6.2) (end -15.5 -10.2)
+      (stroke (width 0.15) (type default)) (layer "Edge.Cuts"))
+    (fp_line (start -15.2 -10.5) (end -8.8 -10.5)
+      (stroke (width 0.15) (type default)) (layer "Edge.Cuts"))
+    (fp_line (start -8.8 6.5) (end -15.2 6.5)
+      (stroke (width 0.15) (type default)) (layer "Edge.Cuts"))
+    (fp_line (start -8.5 -10.2) (end -8.5 6.2)
+      (stroke (width 0.15) (type default)) (layer "Edge.Cuts"))
+    (fp_line (start 8.5 6.2) (end 8.5 -10.2)
+      (stroke (width 0.15) (type default)) (layer "Edge.Cuts"))
+    (fp_line (start 8.8 -10.5) (end 15.2 -10.5)
+      (stroke (width 0.15) (type default)) (layer "Edge.Cuts"))
+    (fp_line (start 15.2 6.5) (end 8.8 6.5)
+      (stroke (width 0.15) (type default)) (layer "Edge.Cuts"))
+    (fp_line (start 15.5 -10.2) (end 15.5 6.2)
+      (stroke (width 0.15) (type default)) (layer "Edge.Cuts"))
+    (fp_arc (start -15.5 -10.2) (mid -15.412132 -10.412132) (end -15.2 -10.5)
+      (stroke (width 0.15) (type default)) (layer "Edge.Cuts"))
+    (fp_arc (start -15.2 6.5) (mid -15.412132 6.412132) (end -15.5 6.2)
+      (stroke (width 0.15) (type default)) (layer "Edge.Cuts"))
+    (fp_arc (start -8.8 -10.5) (mid -8.587868 -10.412132) (end -8.5 -10.2)
+      (stroke (width 0.15) (type default)) (layer "Edge.Cuts"))
+    (fp_arc (start -8.5 6.2) (mid -8.587868 6.412132) (end -8.8 6.5)
+      (stroke (width 0.15) (type default)) (layer "Edge.Cuts"))
+    (fp_arc (start 8.5 -10.2) (mid 8.587868 -10.412132) (end 8.8 -10.5)
+      (stroke (width 0.15) (type default)) (layer "Edge.Cuts"))
+    (fp_arc (start 8.8 6.5) (mid 8.587868 6.412132) (end 8.5 6.2)
+      (stroke (width 0.15) (type default)) (layer "Edge.Cuts"))
+    (fp_arc (start 15.2 -10.5) (mid 15.412132 -10.412132) (end 15.5 -10.2)
+      (stroke (width 0.15) (type default)) (layer "Edge.Cuts"))
+    (fp_arc (start 15.5 6.2) (mid 15.412132 6.412132) (end 15.2 6.5)
       (stroke (width 0.15) (type default)) (layer "Edge.Cuts"))
     (fp_line (start -7 2.525) (end -7 6.875)
@@
     (property "ki_keywords" "switch normally-open pushbutton push-button")
     (attr smd)
-    (fp_text reference "SW5" (at -5.715 8.255) (layer "B.SilkS")
+    (fp_text reference "SW5" (at 3.683 9.525) (layer "B.SilkS")
         (effects (font (size 1 1) (thickness 0.15)) (justify mirror))
     )
@@
     (fp_circle (center 3.25 2.25) (end 1.25 2.5)
       (stroke (width 0.1) (type solid)) (fill none) (layer "F.Fab"))
-    (pad "1" thru_hole circle (at 0 0 90) (size 2 2) (drill 1.1) (layers "*.Cu" "B.Mask")
+    (pad "1" thru_hole circle (at 0 0 90) (size 2 2) (drill 1.1) (layers "*.Cu" "*.Mask")
       (net 1 "RST") (pinfunction "1") (pintype "passive"))
-    (pad "1" thru_hole circle (at 6.5 0 90) (size 2 2) (drill 1.1) (layers "*.Cu" "B.Mask")
+    (pad "1" thru_hole circle (at 6.5 0 90) (size 2 2) (drill 1.1) (layers "*.Cu" "*.Mask")
       (net 1 "RST") (pinfunction "1") (pintype "passive"))
-    (pad "2" thru_hole circle (at 0 4.5 90) (size 2 2) (drill 1.1) (layers "*.Cu" "B.Mask")
+    (pad "2" thru_hole circle (at 0 4.5 90) (size 2 2) (drill 1.1) (layers "*.Cu" "*.Mask")
       (net 2 "GND") (pinfunction "2") (pintype "passive"))
-    (pad "2" thru_hole circle (at 6.5 4.5 90) (size 2 2) (drill 1.1) (layers "*.Cu" "B.Mask")
+    (pad "2" thru_hole circle (at 6.5 4.5 90) (size 2 2) (drill 1.1) (layers "*.Cu" "*.Mask")
       (net 2 "GND") (pinfunction "2") (pintype "passive"))
     (model "${KICAD6_3DMODEL_DIR}/Button_Switch_THT.3dshapes/SW_PUSH_6mm.wrl"
@@
   (gr_line (start 182 133.15) (end 99.545 133.15)
     (stroke (width 0.15) (type default)) (layer "Edge.Cuts"))
-  (gr_text "mfk5 rev. 1 @niw" (at 113.15 130.61) (layer "F.SilkS")
+  (gr_text "mfk5 rev. 2 @niw" (at 113.15 130.61) (layer "F.SilkS")
     (effects (font (size 1 1) (thickness 0.15)))
   )
@@
   (segment (start 137.915 95.05) (end 144.9 95.05) (width 0.25) (layer "F.Cu") (net 3))
   (segment (start 144.9 95.05) (end 146.17 96.32) (width 0.25) (layer "F.Cu") (net 3))
+  (segment (start 148.075 124.26) (end 148.075 113.465) (width 0.25) (layer "F.Cu") (net 3))
   (segment (start 104.26 84.255) (end 102.99 85.525) (width 0.25) (layer "F.Cu") (net 3))
-  (segment (start 148.075 124.26) (end 148.075 114.1) (width 0.25) (layer "F.Cu") (net 3))
   (segment (start 136.645 86.795) (end 136.645 85.525) (width 0.25) (layer "F.Cu") (net 3))
   (segment (start 104.26 90.605) (end 105.53 90.605) (width 0.25) (layer "F.Cu") (net 3))
-  (segment (start 146.17 105.845) (end 146.17 112.195) (width 0.25) (layer "F.Cu") (net 3))
+  (segment (start 146.17 111.56) (end 146.17 105.845) (width 0.25) (layer "F.Cu") (net 3))
   (segment (start 136.645 86.795) (end 136.645 93.78) (width 0.25) (layer "F.Cu") (net 3))
   (segment (start 146.17 96.32) (end 146.17 105.845) (width 0.25) (layer "F.Cu") (net 3))
@@
   (segment (start 135.375 84.255) (end 104.26 84.255) (width 0.25) (layer "F.Cu") (net 3))
   (segment (start 136.645 93.78) (end 137.915 95.05) (width 0.25) (layer "F.Cu") (net 3))
-  (segment (start 148.075 114.1) (end 146.17 112.195) (width 0.25) (layer "F.Cu") (net 3))
+  (segment (start 148.075 113.465) (end 146.17 111.56) (width 0.25) (layer "F.Cu") (net 3))
   (via (at 146.17 105.845) (size 0.8) (drill 0.4) (layers "F.Cu" "B.Cu") (free) (net 3))
   (via (at 136.645 86.795) (size 0.8) (drill 0.4) (layers "F.Cu" "B.Cu") (net 3))
@@
   (segment (start 169.03 96.955) (end 155.06 96.955) (width 0.25) (layer "B.Cu") (net 13))
   (segment (start 106.8 98.225) (end 105.53 98.225) (width 0.25) (layer "B.Cu") (net 13))
-  (segment (start 106.8 100.765) (end 105.53 100.765) (width 0.25) (layer "B.Cu") (net 14))
-  (segment (start 148.075 116.005) (end 149.345 117.275) (width 0.25) (layer "B.Cu") (net 14))
-  (segment (start 146.805 112.83) (end 148.075 114.1) (width 0.25) (layer "B.Cu") (net 14))
-  (segment (start 132.2 99.495) (end 108.07 99.495) (width 0.25) (layer "B.Cu") (net 14))
+  (segment (start 133.47 110.925) (end 134.74 112.195) (width 0.25) (layer "B.Cu") (net 14))
+  (segment (start 148.075 116.132) (end 149.218 117.275) (width 0.25) (layer "B.Cu") (net 14))
+  (segment (start 133.47 100.765) (end 133.47 110.925) (width 0.25) (layer "B.Cu") (net 14))
+  (segment (start 108.07 99.495) (end 132.2 99.495) (width 0.25) (layer "B.Cu") (net 14))
+  (segment (start 148.075 113.465) (end 148.075 116.132) (width 0.25) (layer "B.Cu") (net 14))
+  (segment (start 106.8 100.765) (end 108.07 99.495) (width 0.25) (layer "B.Cu") (net 14))
+  (segment (start 105.53 100.765) (end 106.8 100.765) (width 0.25) (layer "B.Cu") (net 14))
+  (segment (start 146.805 112.195) (end 148.075 113.465) (width 0.25) (layer "B.Cu") (net 14))
   (segment (start 132.2 99.495) (end 133.47 100.765) (width 0.25) (layer "B.Cu") (net 14))
-  (segment (start 133.47 100.765) (end 133.47 111.56) (width 0.25) (layer "B.Cu") (net 14))
-  (segment (start 134.74 112.83) (end 146.805 112.83) (width 0.25) (layer "B.Cu") (net 14))
-  (segment (start 148.075 114.1) (end 148.075 116.005) (width 0.25) (layer "B.Cu") (net 14))
-  (segment (start 133.47 111.56) (end 134.74 112.83) (width 0.25) (layer "B.Cu") (net 14))
-  (segment (start 149.345 117.275) (end 152.775 117.275) (width 0.25) (layer "B.Cu") (net 14))
-  (segment (start 108.07 99.495) (end 106.8 100.765) (width 0.25) (layer "B.Cu") (net 14))
+  (segment (start 134.74 112.195) (end 146.805 112.195) (width 0.25) (layer "B.Cu") (net 14))
+  (segment (start 149.218 117.275) (end 152.775 117.275) (width 0.25) (layer "B.Cu") (net 14))
   (zone (net 2) (net_name "GND") (layer "B.Cu") (hatch edge 0.5)
     (connect_pads (clearance 0.5))
