File: mfk5_top_panel.kicad_pcb (KiCad board)
At the start: 2 copper layers, 57.2 x 57.2 mm, 9 parts

Commit message: Update mfk5 layout.
Changed lines of the file:
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@@
     (fp_line (start -15.25 4.95) (end -15.25 -6.85)
       (stroke (width 0.15) (type default)) (layer "Edge.Cuts"))
-    (fp_line (start -14.95 -7.15) (end -9.05 -7.15)
+    (fp_line (start -14.95 -7.15) (end -13.8 -7.15)
+      (stroke (width 0.15) (type default)) (layer "Edge.Cuts"))
+    (fp_line (start -13.5 -7.45) (end -13.5 -7.85)
+      (stroke (width 0.15) (type default)) (layer "Edge.Cuts"))
+    (fp_line (start -13.2 -8.15) (end -10.8 -8.15)
+      (stroke (width 0.15) (type default)) (layer "Edge.Cuts"))
+    (fp_line (start -10.5 -7.85) (end -10.5 -7.45)
+      (stroke (width 0.15) (type default)) (layer "Edge.Cuts"))
+    (fp_line (start -10.2 -7.15) (end -9.05 -7.15)
       (stroke (width 0.15) (type default)) (layer "Edge.Cuts"))
     (fp_line (start -9.05 5.25) (end -14.95 5.25)
       (stroke (width 0.15) (type default)) (layer "Edge.Cuts"))
-    (fp_line (start -8.75 -6.85) (end -8.75 4.95)
+    (fp_line (start -8.75 -6.85) (end -8.75 -4.3)
       (stroke (width 0.15) (type default)) (layer "Edge.Cuts"))
-    (fp_line (start -7 6.7) (end -7 -6.7)
+    (fp_line (start -8.75 0.3) (end -8.75 4.95)
+      (stroke (width 0.15) (type default)) (layer "Edge.Cuts"))
+    (fp_line (start -8.45 -4) (end -7.3 -4)
+      (stroke (width 0.15) (type default)) (layer "Edge.Cuts"))
+    (fp_line (start -8.45 0) (end -7.3 0)
+      (stroke (width 0.15) (type default)) (layer "Edge.Cuts"))
+    (fp_line (start -7 -4.3) (end -7 -6.7)
+      (stroke (width 0.15) (type default)) (layer "Edge.Cuts"))
+    (fp_line (start -7 6.7) (end -7 0.3)
       (stroke (width 0.15) (type default)) (layer "Edge.Cuts"))
     (fp_line (start -6.7 -7) (end 6.7 -7)
@@
     (fp_line (start 6.7 7) (end -6.7 7)
       (stroke (width 0.15) (type default)) (layer "Edge.Cuts"))
-    (fp_line (start 7 -6.7) (end 7 6.7)
+    (fp_line (start 7 -6.7) (end 7 -4.3)
       (stroke (width 0.15) (type default)) (layer "Edge.Cuts"))
-    (fp_line (start 8.75 4.95) (end 8.75 -6.85)
+    (fp_line (start 7 0.3) (end 7 6.7)
       (stroke (width 0.15) (type default)) (layer "Edge.Cuts"))
-    (fp_line (start 9.05 -7.15) (end 14.95 -7.15)
+    (fp_line (start 7.3 -4) (end 8.45 -4)
+      (stroke (width 0.15) (type default)) (layer "Edge.Cuts"))
+    (fp_line (start 7.3 0) (end 8.45 0)
+      (stroke (width 0.15) (type default)) (layer "Edge.Cuts"))
+    (fp_line (start 8.75 -4.3) (end 8.75 -6.85)
+      (stroke (width 0.15) (type default)) (layer "Edge.Cuts"))
+    (fp_line (start 8.75 4.95) (end 8.75 0.3)
+      (stroke (width 0.15) (type default)) (layer "Edge.Cuts"))
+    (fp_line (start 9.05 -7.15) (end 10.2 -7.15)
+      (stroke (width 0.15) (type default)) (layer "Edge.Cuts"))
+    (fp_line (start 10.5 -7.45) (end 10.5 -7.85)
+      (stroke (width 0.15) (type default)) (layer "Edge.Cuts"))
+    (fp_line (start 10.8 -8.15) (end 13.2 -8.15)
+      (stroke (width 0.15) (type default)) (layer "Edge.Cuts"))
+    (fp_line (start 13.5 -7.85) (end 13.5 -7.45)
+      (stroke (width 0.15) (type default)) (layer "Edge.Cuts"))
+    (fp_line (start 13.8 -7.15) (end 14.95 -7.15)
       (stroke (width 0.15) (type default)) (layer "Edge.Cuts"))
     (fp_line (start 14.95 5.25) (end 9.05 5.25)
@@
     (fp_arc (start -14.95 5.25) (mid -15.162132 5.162132) (end -15.25 4.95)
       (stroke (width 0.15) (type default)) (layer "Edge.Cuts"))
+    (fp_arc (start -13.5 -7.85) (mid -13.412132 -8.062132) (end -13.2 -8.15)
+      (stroke (width 0.15) (type default)) (layer "Edge.Cuts"))
+    (fp_arc (start -13.5 -7.45) (mid -13.587868 -7.237868) (end -13.8 -7.15)
+      (stroke (width 0.15) (type default)) (layer "Edge.Cuts"))
+    (fp_arc (start -10.8 -8.15) (mid -10.587868 -8.062132) (end -10.5 -7.85)
+      (stroke (width 0.15) (type default)) (layer "Edge.Cuts"))
+    (fp_arc (start -10.2 -7.15) (mid -10.412132 -7.237868) (end -10.5 -7.45)
+      (stroke (width 0.15) (type default)) (layer "Edge.Cuts"))
     (fp_arc (start -9.05 -7.15) (mid -8.837868 -7.062132) (end -8.75 -6.85)
+      (stroke (width 0.15) (type default)) (layer "Edge.Cuts"))
+    (fp_arc (start -8.75 0.3) (mid -8.662132 0.087868) (end -8.45 0)
       (stroke (width 0.15) (type default)) (layer "Edge.Cuts"))
     (fp_arc (start -8.75 4.95) (mid -8.837868 5.162132) (end -9.05 5.25)
       (stroke (width 0.15) (type default)) (layer "Edge.Cuts"))
+    (fp_arc (start -8.45 -4) (mid -8.662132 -4.087868) (end -8.75 -4.3)
+      (stroke (width 0.15) (type default)) (layer "Edge.Cuts"))
+    (fp_arc (start -7.3 0) (mid -7.087868 0.087868) (end -7 0.3)
+      (stroke (width 0.15) (type default)) (layer "Edge.Cuts"))
     (fp_arc (start -7 -6.7) (mid -6.912132 -6.912132) (end -6.7 -7)
+      (stroke (width 0.15) (type default)) (layer "Edge.Cuts"))
+    (fp_arc (start -7 -4.3) (mid -7.087868 -4.087868) (end -7.3 -4)
       (stroke (width 0.15) (type default)) (layer "Edge.Cuts"))
     (fp_arc (start -6.7 7) (mid -6.912132 6.912132) (end -7 6.7)
@@
     (fp_arc (start 6.7 -7) (mid 6.912132 -6.912132) (end 7 -6.7)
       (stroke (width 0.15) (type default)) (layer "Edge.Cuts"))
+    (fp_arc (start 7 0.3) (mid 7.087868 0.087868) (end 7.3 0)
+      (stroke (width 0.15) (type default)) (layer "Edge.Cuts"))
     (fp_arc (start 7 6.7) (mid 6.912132 6.912132) (end 6.7 7)
+      (stroke (width 0.15) (type default)) (layer "Edge.Cuts"))
+    (fp_arc (start 7.3 -4) (mid 7.087868 -4.087868) (end 7 -4.3)
+      (stroke (width 0.15) (type default)) (layer "Edge.Cuts"))
+    (fp_arc (start 8.45 0) (mid 8.662132 0.087868) (end 8.75 0.3)
       (stroke (width 0.15) (type default)) (layer "Edge.Cuts"))
     (fp_arc (start 8.75 -6.85) (mid 8.837868 -7.062132) (end 9.05 -7.15)
       (stroke (width 0.15) (type default)) (layer "Edge.Cuts"))
+    (fp_arc (start 8.75 -4.3) (mid 8.662132 -4.087868) (end 8.45 -4)
+      (stroke (width 0.15) (type default)) (layer "Edge.Cuts"))
     (fp_arc (start 9.05 5.25) (mid 8.837868 5.162132) (end 8.75 4.95)
       (stroke (width 0.15) (type default)) (layer "Edge.Cuts"))
+    (fp_arc (start 10.5 -7.85) (mid 10.587868 -8.062132) (end 10.8 -8.15)
+      (stroke (width 0.15) (type default)) (layer "Edge.Cuts"))
+    (fp_arc (start 10.5 -7.45) (mid 10.412132 -7.237868) (end 10.2 -7.15)
+      (stroke (width 0.15) (type default)) (layer "Edge.Cuts"))
+    (fp_arc (start 13.2 -8.15) (mid 13.412132 -8.062132) (end 13.5 -7.85)
+      (stroke (width 0.15) (type default)) (layer "Edge.Cuts"))
+    (fp_arc (start 13.8 -7.15) (mid 13.587868 -7.237868) (end 13.5 -7.45)
+      (stroke (width 0.15) (type default)) (layer "Edge.Cuts"))
     (fp_arc (start 14.95 -7.15) (mid 15.162132 -7.062132) (end 15.25 -6.85)
